File: PCB/KICad-Project/Taupunkt.kicad_sch (KiCad schematic)
At the start: 17 parts, among them J1 DC PWR, J2 AM2302 inside, J3 AM2302 outside, J4 16x4 LCD, J5 D1 MINI - RTC, J6 SD-Card, J7 Relais, SW1 RST, SW2 SW_SPDT_MSM

Commit message: Added BOM, removed backups, updated files
Parts:
- C1: footprint Capacitor_THT:CP_Radial_Tantal_D5.0mm_P5.00mm -> Capacitor_THT:CP_Radial_Tantal_D10.5mm_P5.00mm
- J2: value AM2302 inside -> DHT22 inside
- J3: value AM2302 outside -> DHT22 outside
- J4: value 16x4 LCD -> 20x4 LCD
- J7: value Relais -> Relay Fan1
- R1, R2, R3, R4, R5: footprint Resistor_THT:R_Axial_DIN0204_L3.6mm_D1.6mm_P5.08mm_Horizontal -> Resistor_THT:R_Axial_DIN0207_L6.3mm_D2.5mm_P7.62mm_Horizontal
- SW1: value RST -> RST-Switch
- SW2: value SW_SPDT_MSM -> ModeSwitch
Connections:
- net GND is gone; now on an unnamed net: A1.29 (GND), C1.2, C2.2, J1.1 (Pin_1), J2.1 (Pin_1), J3.1 (Pin_1), J4.3 (Pin_3), J5.7 (Pin_7), J6.6 (Pin_6), J7.1 (Pin_1), SW1.2, SW2.1
- net RelSwitch: no longer A1.9 (D6), R5.2
- new net RelSwitchCtrl: A1.9 (D6), R5.2
Other:
- moved on the sheet: J4
